Commit message: Added funky models and did write-up in calculations doc

File: projects/02_segbot/urdf/segbot.urdf (robot description, URDF)
Before this commit: robot platform, 3 links, 2 joints
Links:
- link chassis: geometry collision box size=0.4 0.6 0.8; visual mesh filename=Bullet_Bill.stl scale=0.001 0.001 0.001

File: projects/02_segbot/urdf/segbot2.urdf (robot description, URDF)
Before this commit: robot platform, 3 links, 2 joints
Links:
- link chassis: geometry collision box size=0.4 0.6 0.8; visual mesh filename=Kart-HP.stl scale=0.3 0.3 0.3
